Commit message: feat: apply measured calibration offsets to so101 urdf joint origins
Rotate the origin of three joints about their axis so the model
matches the real arm at the LeRobot-calibrated zero, measured with a
phone level on 2026-09-27: shoulder_lift +4.7 deg, elbow_flex +12.6 deg,
gripper +39.7 deg (closed reads -0.867 rad while the URDF jaws touch at
-0.1745 rad, because LeRobot homes the gripper at mid-range). Only the
rpy attributes change; xyz, limits, meshes and the other joints stay as
in the upstream file. Verified with check_urdf, mesh principal-axis
angles (6.4 / 23.7 deg vs measured 7.4 / 22.8) and jaw contact at the
measured closed reading.

File: Studies/Hardware-Arm/stage1/ros2_pkg/so101_description/urdf/so101.urdf.xacro (robot description, xacro)
@@ -10,6 +10,6 @@
     3. ROS 1 형식 <transmission> 블록 6개 제거 (ros2_control 은 쓰지 않는다)
     4. 파일 끝에 <ros2_control> 블록 추가
-  link / joint 의 수치 (origin, inertia, limit) 는 원본 그대로다.
-  캘리브 오프셋 반영은 Stage 1 W4 에서 한다 (URDF_guide.md 0절).
+    5. W4 캘리브 오프셋 (2026-09-27): shoulder_lift · elbow_flex · gripper 의 joint origin rpy 를 실물 영점에 맞춰 회전
+       (각 joint 의 주석과 URDF_guide.md 5절). 그 밖의 link / joint 수치 (xyz, inertia, limit) 는 원본 그대로다.
 -->
 <!-- Generated using onshape-to-robot -->
@@ -334,5 +334,8 @@
   <!-- Joint from gripper to moving_jaw_so101_v1 -->
   <joint name="gripper" type="revolute">
-    <origin xyz="0.0202 0.0188 -0.0234" rpy="1.5708 -5.24284e-08 -1.41553e-15"/>
+    <!-- W4 캘리브 오프셋 보정 (2026-09-27): 관절축 둘레 +39.7도 (+0.6925 rad). 원본 rpy 는 1.5708 0 0.
+       LeRobot 캘리브레이션은 그리퍼도 가동 범위 가운데를 서보 0 으로 두어, 실물 닫힘이 -0.867 rad 로 읽힌다.
+       URDF 에서 조가 닿는 각도는 하한 -0.1745 rad 이므로 그 차이만큼 돌린다. -->
+    <origin xyz="0.0202 0.0188 -0.0234" rpy="1.57080 -0.69250 -0.00000"/>
     <parent link="gripper_link"/>
     <child link="moving_jaw_so101_v1_link"/>
@@ -359,5 +362,7 @@
   <!-- Note: 5-degree calibration offset applied to joint limits -->
   <joint name="elbow_flex" type="revolute">
-    <origin xyz="-0.11257 -0.028 1.73763e-16" rpy="-3.63608e-16 8.74301e-16 1.5708"/>
+    <!-- W4 캘리브 오프셋 보정 (2026-09-27): 관절축 둘레 +12.6도 (+0.21991 rad). 원본 rpy 는 0 0 1.5708.
+       영점 자세에서 실물 아래팔이 수평보다 22.8도 아래였고 (위팔 기울기 7.4도 포함) 그때 관절값이 +2.8도였다. -->
+    <origin xyz="-0.11257 -0.028 1.73763e-16" rpy="0 0 1.79071"/>
     <parent link="upper_arm_link"/>
     <child link="lower_arm_link"/>
@@ -367,5 +372,7 @@
   <!-- Joint from shoulder to upper_arm -->
   <joint name="shoulder_lift" type="revolute">
-    <origin xyz="-0.0303992 -0.0182778 -0.0542" rpy="-1.5708 -1.5708 0"/>
+    <!-- W4 캘리브 오프셋 보정 (2026-09-27): 관절축 둘레 +4.7도 (+0.08203 rad). 원본 rpy 는 -1.5708 -1.5708 0.
+       영점 자세에서 실물 위팔이 수직보다 앞으로 7.4도 기울어 있었고 그때 관절값이 +2.7도였다. -->
+    <origin xyz="-0.0303992 -0.0182778 -0.0542" rpy="-1.5708 -1.48877 0"/>
     <parent link="shoulder_link"/>
     <child link="upper_arm_link"/>

Commit message: feat: enable ros2_control command limits with calibrated joint ranges
Set enforce_command_limits: true on the controller manager (Jazzy
defaults to off) and replace the URDF limit lower/upper of five joints
with the LeRobot calibration ranges converted to radians, 0.02 rad
inside; wrist_roll keeps the upstream values because it is not
calibrated. The upstream limits did not cover the real arm (rest pose
shoulder_lift -1.772, gripper closed -0.867). Verified on the mock
hardware: commands of +3.0 / -3.0 on shoulder_pan and -3.0 on gripper
are clamped to 1.700 / -1.695 / -0.845 and the log reports enforcement
enabled. Original limit lines are kept as comments next to each joint.

File: Studies/Hardware-Arm/stage1/ros2_pkg/so101_description/urdf/so101.urdf.xacro (robot description, xacro)
@@ -11,5 +11,8 @@
     4. 파일 끝에 <ros2_control> 블록 추가
     5. W4 캘리브 오프셋 (2026-09-27): shoulder_lift · elbow_flex · gripper 의 joint origin rpy 를 실물 영점에 맞춰 회전
-       (각 joint 의 주석과 URDF_guide.md 5절). 그 밖의 link / joint 수치 (xyz, inertia, limit) 는 원본 그대로다.
+       (각 joint 의 주석과 URDF_guide.md 5절)
+    6. W5 소프트 리밋 (2026-09-30): wrist_roll 을 뺀 joint 5개의 <limit lower/upper> 를 LeRobot 캘리브 파일의
+       실물 범위 안쪽 0.02 rad 로 교체 (ros2_driver_setup.md 6.2절). 원본 값은 각 joint 의 주석에 남겼다.
+  그 밖의 link / joint 수치 (xyz, inertia, effort, velocity) 는 원본 그대로다.
 -->
 <!-- Generated using onshape-to-robot -->
@@ -341,5 +344,8 @@
     <child link="moving_jaw_so101_v1_link"/>
     <axis xyz="0 0 1"/>
+    <!--
     <limit effort="10" velocity="10" lower="-0.174533" upper="1.74533"/>
+    -->
+    <limit effort="10" velocity="10" lower="-0.845" upper="1.462"/>
   </joint>
   <!-- Joint from wrist to gripper -->
@@ -357,5 +363,8 @@
     <child link="wrist_link"/>
     <axis xyz="0 0 1"/>
+    <!--
     <limit effort="10" velocity="10" lower="-1.65806" upper="1.65806"/>
+    -->
+    <limit effort="10" velocity="10" lower="-1.686" upper="1.816"/>
   </joint>
   <!-- Joint from upper_arm to lower_arm -->
@@ -368,5 +377,8 @@
     <child link="lower_arm_link"/>
     <axis xyz="0 0 1"/>
+    <!--
     <limit effort="10" velocity="10" lower="-1.69" upper="1.69"/>
+    -->
+    <limit effort="10" velocity="10" lower="-2.019" upper="1.529"/>
   </joint>
   <!-- Joint from shoulder to upper_arm -->
@@ -378,5 +390,8 @@
     <child link="upper_arm_link"/>
     <axis xyz="0 0 1"/>
+    <!--
     <limit effort="10" velocity="10" lower="-1.74533" upper="1.74533"/>
+    -->
+    <limit effort="10" velocity="10" lower="-1.822" upper="1.787"/>
   </joint>
   <!-- Joint from base to shoulder -->
@@ -386,5 +401,8 @@
     <child link="shoulder_link"/>
     <axis xyz="0 0 1"/>
+    <!--
     <limit effort="10" velocity="10" lower="-1.91986" upper="1.91986"/>
+    -->
+    <limit effort="10" velocity="10" lower="-1.695" upper="1.700"/>
   </joint>
   <!--

Commit message: fix: widen soft limits to 0.05 rad outside the calibrated range
The first values sat 0.02 rad inside the calibration range, but the
real arm goes slightly past the recorded extremes at its mechanical
stops (rest pose elbow_flex 1.542-1.555 vs calibrated max 1.549,
gripper closed -0.867 vs min -0.865). The Jazzy joint limiter throws
when the actual position is outside the limits, which killed
ros2_control_node at bringup. Limits are now calibration +-0.05 rad
for the five calibrated joints; wrist_roll keeps upstream values.
Verified: bringup on the real arm starts clean at rest, +0.05 rad
commands behave as before, hold commands are not clamped.

File: Studies/Hardware-Arm/stage1/ros2_pkg/so101_description/urdf/so101.urdf.xacro (robot description, xacro)
@@ -347,5 +347,5 @@
     <limit effort="10" velocity="10" lower="-0.174533" upper="1.74533"/>
     -->
-    <limit effort="10" velocity="10" lower="-0.845" upper="1.462"/>
+    <limit effort="10" velocity="10" lower="-0.915" upper="1.532"/>
   </joint>
   <!-- Joint from wrist to gripper -->
@@ -366,5 +366,5 @@
     <limit effort="10" velocity="10" lower="-1.65806" upper="1.65806"/>
     -->
-    <limit effort="10" velocity="10" lower="-1.686" upper="1.816"/>
+    <limit effort="10" velocity="10" lower="-1.756" upper="1.886"/>
   </joint>
   <!-- Joint from upper_arm to lower_arm -->
@@ -380,5 +380,5 @@
     <limit effort="10" velocity="10" lower="-1.69" upper="1.69"/>
     -->
-    <limit effort="10" velocity="10" lower="-2.019" upper="1.529"/>
+    <limit effort="10" velocity="10" lower="-2.089" upper="1.599"/>
   </joint>
   <!-- Joint from shoulder to upper_arm -->
@@ -393,5 +393,5 @@
     <limit effort="10" velocity="10" lower="-1.74533" upper="1.74533"/>
     -->
-    <limit effort="10" velocity="10" lower="-1.822" upper="1.787"/>
+    <limit effort="10" velocity="10" lower="-1.892" upper="1.857"/>
   </joint>
   <!-- Joint from base to shoulder -->
@@ -404,5 +404,5 @@
     <limit effort="10" velocity="10" lower="-1.91986" upper="1.91986"/>
     -->
-    <limit effort="10" velocity="10" lower="-1.695" upper="1.700"/>
+    <limit effort="10" velocity="10" lower="-1.765" upper="1.770"/>
   </joint>
   <!--
